Commit message: Readme changes and other tweaks

File: src/robot_configs/franka_panda_config/config/franka_panda.urdf (robot description, URDF)
Before this commit: robot franka_panda, 14 links, 13 joints
Joints:
- joint end_effector_frame_fixed_joint: origin xyz=0 0 0.21 rpy=3.14159 -1.57079 -0.785398163397 -> xyz=0 0 0.1 rpy=0 0 0; parent panda_link7 -> panda_hand

File: src/robot_configs/kinova_config/config/kinova.urdf (robot description, URDF)
Before this commit: robot kinova, 15 links, 14 joints
Joints:
- joint j2s6s200_joint_end_effector: limit lower=0 upper=0 effort=2000 velocity=1 -> lower=0 upper=0 effort=2000 velocity=0.99
- joint j2s6s200_joint_finger_1: limit lower=0 upper=1.51 effort=2 velocity=1 -> lower=0 upper=1.51 effort=2 velocity=0.99
- joint j2s6s200_joint_finger_2: limit lower=0 upper=1.51 effort=2 velocity=1 -> lower=0 upper=1.51 effort=2 velocity=0.99
- joint j2s6s200_joint_finger_tip_1: limit lower=0 upper=2 effort=2 velocity=1 -> lower=0 upper=2 effort=2 velocity=0.99
- joint j2s6s200_joint_finger_tip_2: limit lower=0 upper=2 effort=2 velocity=1 -> lower=0 upper=2 effort=2 velocity=0.99
